File: USBTTLPGM_00.kicad_sch (KiCad schematic)
At the start: 29 parts, among them CN1 +5V, CN2 D-, CN3 D+, CN4 GND, IC1 LR6207, IC2 CH340C, P1 Boot, P2 RST, P3 GND, P4 Rx, P5 Tx, P6 +3Vout, SW1 B3S-1000

Commit message: .
Parts:
- C1: symbol Capacitor_Tantal_0805_6.3V_10perc_AVX:4u7, SMD 0805, 6.3V, 10%, AVX -> Capacitor_Tantal_SMD_0805_6.3V_10perc_AVX:4u7, SMD 0805, 6.3V, 10%
- C2: value 100n -> 100n/50V; symbol Capacitor_Ceramic_0805_50V_X7R_Generic:100n, SMD 0805, 50V, X7R -> Capacitor_Ceramic_SMD_0805_50V_X7R_Generic:100n, SMD 0805, 50V, X7R
- CN1: value +5V -> TestPoint
- CN2: value D- -> TestPoint
- CN3: value D+ -> TestPoint
- CN4, P3: value GND -> TestPoint
- LD3: value KP-2012MGC-Green -> KP-2012QBC-D-Blue
- LD4: Z-SYSCODE 491 -> 10692
- P1: value Boot -> TestPoint
- P2: value RST -> TestPoint
- P4: value Rx -> TestPoint
- P5: value Tx -> TestPoint
- P6: value +3Vout -> TestPoint
- R1: value 10k 5% -> 10k
- R10, R2, R3, R8, R9: value 2k2 5% -> 2k2
